File: Hardware/Sergej_H00/Motors.sch (KiCad schematic (older format))
At the start: 52 parts, among them J10 Conn_01x02, J11 Conn_01x02, J12 Conn_01x03_Male, J13 Conn_01x02, J14 Conn_01x02, J15 Conn_01x03_Male, J7 Conn_01x02, J8 Conn_01x03_Male, J9 Conn_01x02, Q6 AO3400A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

Commit message: updated schematics - part values and LCSC numbers
Parts:
- Q6, Q7, Q8, Q9: LCSC (none) -> C20917
Changed lines of the file:
@@
 F 2 "Package_TO_SOT_SMD:SOT-23" H 7900 4400 50  0001 C CNN
 F 3 "~" H 7700 4300 50  0001 C CNN
+F 4 "C20917" H 7700 4300 50  0001 C CNN "LCSC"
 	1    7700 4300
 	1    0    0    -1
@@
 F 2 "Package_TO_SOT_SMD:SOT-23" H 7900 6100 50  0001 C CNN
 F 3 "~" H 7700 6000 50  0001 C CNN
+F 4 "C20917" H 7700 6000 50  0001 C CNN "LCSC"
 	1    7700 6000
 	1    0    0    -1
@@
 F 2 "Package_TO_SOT_SMD:SOT-23" H 9900 4400 50  0001 C CNN
 F 3 "~" H 9700 4300 50  0001 C CNN
+F 4 "C20917" H 9700 4300 50  0001 C CNN "LCSC"
 	1    9700 4300
 	1    0    0    -1
@@
 F 2 "Package_TO_SOT_SMD:SOT-23" H 9900 6100 50  0001 C CNN
 F 3 "~" H 9700 6000 50  0001 C CNN
+F 4 "C20917" H 9700 6000 50  0001 C CNN "LCSC"
 	1    9700 6000
 	1    0    0    -1
