File: Hardware/Sergej_H00/Mux Demux Matrix.sch (KiCad schematic (older format))
At the start: 23 parts, among them U13 74HC595, U14 74HC595, U15 CD4051B, U20 74HC595, U21 74HC595

Commit message: updated schematics - part values and LCSC numbers
Parts:
- R42, R43: LCSC (none) -> C22962
Changed lines of the file:
@@
 F 2 "Resistor_SMD:R_0603_1608Metric" V 4130 2250 50  0001 C CNN
 F 3 "~" H 4200 2250 50  0001 C CNN
+F 4 "C22962" H 4200 2250 50  0001 C CNN "LCSC"
 	1    4200 2250
 	0    1    1    0
@@
 F 2 "Resistor_SMD:R_0603_1608Metric" V 4130 2550 50  0001 C CNN
 F 3 "~" H 4200 2550 50  0001 C CNN
+F 4 "C22962" H 4200 2550 50  0001 C CNN "LCSC"
 	1    4200 2550
 	0    1    1    0
