File: Hardware/Sergej_H00/Power.sch (KiCad schematic (older format))
At the start: 48 parts, among them IC1 TP4056, J16 Conn_01x02_Male, Q5 S8050, SW3 MT-102, U4 AMS1117-3.3, U5 TPS61088RHLR, U6 MT3608

Commit message: updated schematics - part values and LCSC numbers
Parts:
- C39: value more than 1uF, footprint? -> 1u; LCSC (none) -> C15849
- C41: value f -> 1n; LCSC (none) -> C1588
- F1: value Fuse -> Fuse 15A
- IC1: LCSC (none) -> C16581
- R15: value R -> 24K; LCSC (none) -> C23352
- R16: value R -> 150K; LCSC (none) -> C22807
- R17: value R -> 270K; LCSC (none) -> C22965
- R18: value R -> 240K; LCSC (none) -> C4197
- R19, R28: value R -> 30K; LCSC (none) -> C22984
- R23: value 3M3 -> 3M; LCSC (none) -> C23156
- R26: LCSC (none) -> C7250
- R27: value R -> 220K; LCSC (none) -> C22961
Changed lines of the file:
@@
 AR Path="/600F65F0/60102113" Ref="F1"  Part="1"
 F 0 "F1" H 9960 4996 50  0000 L CNN
-F 1 "Fuse" H 9960 4905 50  0000 L CNN
+F 1 "Fuse 15A" H 9960 4905 50  0000 L CNN
 F 2 "Fuse:Fuse_1206_3216Metric" V 9830 4950 50  0001 C CNN
 F 3 "~" H 9900 4950 50  0001 C CNN
@@
 P 2350 1950
 F 0 "R18" H 2420 1996 50  0000 L CNN
-F 1 "R" H 2420 1905 50  0000 L CNN
+F 1 "240K" H 2420 1905 50  0000 L CNN
 F 2 "Resistor_SMD:R_0603_1608Metric" V 2280 1950 50  0001 C CNN
 F 3 "~" H 2350 1950 50  0001 C CNN
+F 4 "C4197" H 2350 1950 50  0001 C CNN "LCSC"
 	1    2350 1950
 	1    0    0    -1
@@
 P 5450 1550
 F 0 "R15" V 5243 1550 50  0000 C CNN
-F 1 "R" V 5334 1550 50  0000 C CNN
+F 1 "24K" V 5334 1550 50  0000 C CNN
 F 2 "Resistor_SMD:R_0603_1608Metric" V 5380 1550 50  0001 C CNN
 F 3 "~" H 5450 1550 50  0001 C CNN
+F 4 "C23352" H 5450 1550 50  0001 C CNN "LCSC"
 	1    5450 1550
 	0    1    1    0
@@
 P 5750 1550
 F 0 "C41" V 5498 1550 50  0000 C CNN
-F 1 "f" V 5589 1550 50  0000 C CNN
+F 1 "1n" V 5589 1550 50  0000 C CNN
 F 2 "Capacitor_SMD:C_0603_1608Metric" H 5788 1400 50  0001 C CNN
 F 3 "~" H 5750 1550 50  0001 C CNN
+F 4 "C1588" H 5750 1550 50  0001 C CNN "LCSC"
 	1    5750 1550
 	0    1    1    0
@@
 P 4650 950
 F 0 "C39" V 4398 950 50  0000 C CNN
-F 1 "more than 1uF, footprint?" V 4489 950 50  0000 C CNN
+F 1 "1u" V 4489 950 50  0000 C CNN
 F 2 "Capacitor_SMD:C_0603_1608Metric" H 4688 800 50  0001 C CNN
 F 3 "~" H 4650 950 50  0001 C CNN
+F 4 "C15849" H 4650 950 50  0001 C CNN "LCSC"
 	1    4650 950
 	0    1    1    0
@@
 P 4750 1750
 F 0 "R16" V 4650 1650 50  0000 C CNN
-F 1 "R" V 4634 1750 50  0000 C CNN
+F 1 "150K" V 4634 1750 50  0000 C CNN
 F 2 "Resistor_SMD:R_0603_1608Metric" V 4680 1750 50  0001 C CNN
 F 3 "~" H 4750 1750 50  0001 C CNN
+F 4 "C22807" H 4750 1750 50  0001 C CNN "LCSC"
 	1    4750 1750
 	0    1    1    0
@@
 F 2 "Package_SO:SOIC-8-1EP_3.9x4.9mm_P1.27mm_EP2.514x3.2mm_ThermalVias" H 8650 5050 50  0001 L BNN
 F 3 "" H 8650 5050 50  0001 C CNN
+F 4 "C16581" H 8650 5050 50  0001 C CNN "LCSC"
 	1    8650 5050
 	1    0    0    -1
@@
 F 2 "Resistor_SMD:R_0603_1608Metric" V 2030 5450 50  0001 C CNN
 F 3 "~" H 2100 5450 50  0001 C CNN
+F 4 "C7250" H 2100 5450 50  0001 C CNN "LCSC"
 	1    2100 5450
 	-1   0    0    1
@@
 P 6200 1750
 F 0 "R17" V 6100 1650 50  0000 C CNN
-F 1 "R" V 6084 1750 50  0000 C CNN
+F 1 "270K" V 6084 1750 50  0000 C CNN
 F 2 "Resistor_SMD:R_0603_1608Metric" V 6130 1750 50  0001 C CNN
 F 3 "~" H 6200 1750 50  0001 C CNN
+F 4 "C22965" H 6200 1750 50  0001 C CNN "LCSC"
 	1    6200 1750
 	-1   0    0    1
@@
 P 6200 2550
 F 0 "R19" V 6100 2450 50  0000 C CNN
-F 1 "R" V 6084 2550 50  0000 C CNN
+F 1 "30K" V 6084 2550 50  0000 C CNN
 F 2 "Resistor_SMD:R_0603_1608Metric" V 6130 2550 50  0001 C CNN
 F 3 "~" H 6200 2550 50  0001 C CNN
+F 4 "C22984" H 6200 2550 50  0001 C CNN "LCSC"
 	1    6200 2550
 	-1   0    0    1
@@
 P 4550 5700
 F 0 "R27" V 4450 5600 50  0000 C CNN
-F 1 "R" V 4434 5700 50  0000 C CNN
+F 1 "220K" V 4434 5700 50  0000 C CNN
 F 2 "Resistor_SMD:R_0603_1608Metric" V 4480 5700 50  0001 C CNN
 F 3 "~" H 4550 5700 50  0001 C CNN
+F 4 "C22961" H 4550 5700 50  0001 C CNN "LCSC"
 	1    4550 5700
 	-1   0    0    1
@@
 P 4550 6150
 F 0 "R28" V 4450 6050 50  0000 C CNN
-F 1 "R" V 4434 6150 50  0000 C CNN
+F 1 "30K" V 4434 6150 50  0000 C CNN
 F 2 "Resistor_SMD:R_0603_1608Metric" V 4480 6150 50  0001 C CNN
 F 3 "~" H 4550 6150 50  0001 C CNN
+F 4 "C22984" H 4550 6150 50  0001 C CNN "LCSC"
 	1    4550 6150
 	-1   0    0    1
@@
 P 10500 5350
 F 0 "R23" H 10570 5396 50  0000 L CNN
-F 1 "3M3" H 10570 5305 50  0000 L CNN
+F 1 "3M" H 10570 5305 50  0000 L CNN
 F 2 "Resistor_SMD:R_0603_1608Metric" V 10430 5350 50  0001 C CNN
 F 3 "~" H 10500 5350 50  0001 C CNN
+F 4 "C23156" H 10500 5350 50  0001 C CNN "LCSC"
 	1    10500 5350
 	1    0    0    -1
