File: Hardware/Sergej_H00/Sergej_H00.kicad_pcb (KiCad board)
At the start: 2 copper layers, 90 x 100 mm, 203 parts, among them IC1 TP4056, J1 Conn_01x06_Female, J10 Conn_01x02, J11 Conn_01x02, J12 Conn_01x03_Male, J13 Conn_01x02, J14 Conn_01x02, J15 Conn_01x03_Male, J16 Conn_01x02_Male, J2 Conn_01x06_Female, J3 Conn_01x05_Male, J4 Conn_01x05_Male, J5 TYPE-C-31-M-12, J6 Conn_01x01_Male, J7 Conn_01x02, J8 Conn_01x03_Male, J9 Conn_01x02, Q1 2N7002, Q2 S8050, Q3 S8050, Q5 S8050, Q6 AO3400A, Q7 AO3400A, Q8 AO3400A, Q9 AO3400A, SW1 Rotary_Encoder_Switch, SW2 SW_DPST, SW3 MT-102, U1 ESP32-WROOM-32D, U10 TCRT5000, U11 TCRT5000, U12 TCRT5000, U13 74HC595, U14 74HC595, U15 CD4051B, U16 DRV8871DDA, U17 LM358, U18 DRV8871DDA, U19 LM358, U2 MPU-6050, U20 74HC595, U21 74HC595, U3 CH340G, U4 AMS1117-3.3, U5 TPS61088RHLR, U6 MT3608, U7 TCRT5000, U8 TCRT5000, U9 TCRT5000, Y1 12MHz

Commit message: Routed PCB
Parts:
- added .: ., Sergej_Library:Vedatori_15mm, F.Cu at (63.4, 96.0)
Connections:
- J5 pad S1: GND -> Net-(J5-PadS1)
Routing:
- net +3V3: track 102.3 -> 389.0 mm, vias 0 -> 10
- net +5V: track 112.3 -> 312.4 mm, vias 2 -> 9
- net /Mux Demux Matrix/REG_OE: track 0.00 -> 179.4 mm, vias 0 -> 14
- net /Mux Demux Matrix/REG_LAT: track 0.00 -> 153.0 mm, vias 0 -> 8
- net /Mux Demux Matrix/Analog_MUX: track 0.00 -> 147.1 mm, vias 0 -> 14
- net /Mux Demux Matrix/Analog_IN_7: track 3.08 -> 145.8 mm, vias 0 -> 4
- net /Mux Demux Matrix/REG_CLK: track 0.00 -> 139.0 mm, vias 0 -> 10
- net /Motors/SERVO1_CURRENT: track 0.00 -> 119.9 mm, vias 0 -> 10
- net Net-(R40-Pad2): track 1.52 -> 120.2 mm, vias 0 -> 7
- net Net-(R38-Pad2): track 1.52 -> 118.9 mm, vias 0 -> 7
- net /Motors/MOTB_IN1: track 0.00 -> 114.1 mm, vias 0 -> 6
- net /Motors/SERVO2_CURRENT: track 0.00 -> 105.8 mm, vias 0 -> 10
- net /Mux Demux Matrix/REG_DAT: track 0.00 -> 105.6 mm, vias 0 -> 10
- net /Power/5V_ENABLE: track 7.56 -> 108.6 mm, vias 0 -> 4
- net SDA: track 20.0 -> 119.9 mm, vias 0 -> 4
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Other:
- board text added: "+ - MOT1"
- board text added: "+ - MOT2"
- board text added: "+ - MOT3"
- board text added: "+ - MOT4"
- board text added: "3V3 GND SCL SDA GPIO1 XSHUT"
- board text added: "5V GND"
- board text added: "FULL CHARGING"
- board text added: "GND 5V PWM"
- board text added: "LIDAR 1 LIDAR 2"
- board text added: "MOTA"
- board text added: "MOTB"
- board text added: "SDA SCL 5V 3V3 GND"
- board text added: "SERGEJ_H00"
- board text added: "SERVO 1 SERVO 2 SERVO 3"
- board text added: "TOUCH"

Commit message: Final changes made to Sergej_H00, exported gerbers
Parts:
- added G***: LOGO, 0Logo:Coufal_elektronika_text_30x13mm, B.Cu at (44.5, 15.6)
Other:
- board text added: "+ - MOT 2"
- board text added: "+ - MOT 3"
- board text added: "+ - MOT 4"
- board text added: "+ - MOT 5"
- board text added: "12V 5V"
- board text added: "MOT 0"
- board text added: "MOT 1"
- board text added: "Sergej project designed with passion by the Vědátoři team 03-2021"
- board text removed: "+ - MOT1"
- board text removed: "+ - MOT2"
- board text removed: "+ - MOT3"
- board text removed: "+ - MOT4"
- board text removed: "MOTA"
- board text removed: "MOTB"
