File: Hardware/Sergej_H00/USB.sch (KiCad schematic (older format))
At the start: 17 parts, among them J5 TYPE-C-31-M-12, Q2 S8050, Q3 S8050, U3 CH340G, Y1 12MHz

Commit message: Routed PCB
Connections:
- net GND: no longer J5.S1 (SHIELD)
- no-connect marks 5 -> 6
Changed lines of the file:
@@
-	1    0    0    -1
-$EndComp
-$Comp
-L power:GND #PWR?
-U 1 1 601A619F
-P 3300 4350
-AR Path="/60171EF5/601A619F" Ref="#PWR?"  Part="1"
-AR Path="/6018ABDD/601A619F" Ref="#PWR050"  Part="1"
-F 0 "#PWR050" H 3300 4100 50  0001 C CNN
-F 1 "GND" H 3305 4177 50  0000 C CNN
-F 2 "" H 3300 4350 50  0001 C CNN
-F 3 "" H 3300 4350 50  0001 C CNN
-	1    3300 4350
 	1    0    0    -1
 $EndComp
@@
 Wire Wire Line
 	4200 3100 4200 3050
+NoConn ~ 3300 4350
 $EndSCHEMATC

Commit message: Notes for H01 and electronics analysis.
Parts:
- C12, C13: LCSC C84711 -> C1653
Changed lines of the file:
@@
 F 2 "Capacitor_SMD:C_0603_1608Metric" H 5088 4000 50  0001 C CNN
 F 3 "~" H 5050 4150 50  0001 C CNN
-F 4 "C84711" H 5050 4150 50  0001 C CNN "LCSC"
+F 4 "C1653" H 5050 4150 50  0001 C CNN "LCSC"
 	1    5050 4150
 	1    0    0    -1
@@
 F 2 "Capacitor_SMD:C_0603_1608Metric" H 5488 4000 50  0001 C CNN
 F 3 "~" H 5450 4150 50  0001 C CNN
-F 4 "C84711" H 5450 4150 50  0001 C CNN "LCSC"
+F 4 "C1653" H 5450 4150 50  0001 C CNN "LCSC"
 	1    5450 4150
 	1    0    0    -1
