File: Hardware/TrackJet_H01/Power.sch (KiCad schematic (older format))
At the start: 48 parts, among them IC1 TP4056, J16 Conn_01x02_Male, Q5 S8050, SW3 MT-102, U4 AMS1117-3.3, U5 TPS61088RHLR, U6 MT3608

Commit message: Updated H01 PCB
Parts:
- removed C58: 100n, Capacitor_SMD:C_0603_1608Metric, symbol Device:C
- removed Q5: S8050, Package_TO_SOT_SMD:SOT-23, symbol Device:Q_NPN_BEC
- removed R24: 51K, Resistor_SMD:R_0603_1608Metric, symbol Device:R
- added D14: LED_GREEN, LED_THT:LED_D3.0mm, symbol Device:LED
- added D15: B5819W, Diode_SMD:D_SOD-123, symbol Device:D_Schottky
- IC1: LCSC C16581 -> C382139
- R17: value 270K -> 200K; LCSC C22965 -> C25811
- R26: value 10M -> 1K; LCSC C7250 -> C21190
Connections:
- net 5V_ENABLE is gone; now on net +5V: R26.1
- net +BATT: now also U6.4 (EN); no longer R26.2
- net GND: now also D14.1 (K), D15.2 (A)
- net at F1.1, IC1.5 (BAT), SW3.2 (B): now also D15.1 (K)
- new net: D14.2 (A), R26.2
Other:
- moved on the sheet: C54, C55, C56, C57, D12, L2, R27, R28, U6
