File: Hardware/TrackJet_H01/TrackJet_H01_before_autoroute.kicad_pcb (KiCad board)
At the start: 2 copper layers, 90 x 100 mm, 205 parts, among them IC1 TP4056, J1 Conn_01x06_Female, J10 Conn_01x02, J11 Conn_01x02, J12 Conn_01x03_Male, J13 Conn_01x02, J14 Conn_01x02, J15 Conn_01x03_Male, J16 Conn_01x02_Male, J2 Conn_01x06_Female, J3 Conn_01x05_Male, J4 Conn_01x05_Male, J5 TYPE-C-31-M-12, J6 Conn_01x01_Male, J7 Conn_01x02, J8 Conn_01x03_Male, J9 Conn_01x02, Q1 2N7002, Q2 S8050, Q3 S8050, Q6 AO3400A, Q7 AO3400A, Q8 AO3400A, Q9 AO3400A, SW1 Rotary_Encoder_Switch, SW2 SW_DPST, SW3 MT-102, U1 ESP32-WROOM-32D, U10 TCRT5000, U11 TCRT5000, U12 TCRT5000, U13 74HC595, U14 74HC595, U15 CD4051B, U16 DRV8871DDA, U17 LM358, U18 DRV8871DDA, U19 LM358, U2 MPU-6050, U20 74HC595, U21 74HC595, U3 CH340G, U4 AMS1117-3.3, U5 TPS61088RHLR, U6 MT3608, U7 TCRT5000, U8 TCRT5000, U9 TCRT5000, Y1 12MHz

Commit message: Updated H01 PCB
Parts:
- turned C20 to 180 degrees
Routing:
- net /Encoders/ENCODER6: track 111.7 -> 0.00 mm, vias 6 -> 0
- net /Motors/SERVO3_CTRL: track 85.7 -> 0.00 mm, vias 10 -> 0
- net /Encoders/ENCODER5: track 76.9 -> 0.00 mm, vias 6 -> 0
- net /Encoders/ENCODER4: track 70.5 -> 0.00 mm, vias 12 -> 0
- net /Encoders/ENCODER2: track 67.7 -> 0.00 mm, vias 8 -> 0
- net +3V3: track 441.9 -> 379.0 mm, vias 16 -> 10
- net /Motors/SERVO2_CURRENT: track 0.00 -> 45.3 mm, vias 0 -> 6
- net /Power/5V_ENABLE: track 0.00 -> 43.6 mm, vias 0 -> 3
- net /Motors/SERVO1_CURRENT: track 0.00 -> 41.4 mm, vias 0 -> 6
- net /Mux Demux Matrix/Analog_IN_6: track 36.0 -> 0.00 mm, vias 4 -> 0
- net /Mux Demux Matrix/Analog_IN_4: track 33.4 -> 0.00 mm, vias 4 -> 0
- net /Motors/SERVO2_CTRL: track 118.8 -> 87.2 mm, vias 4 -> 1
- net Net-(R34-Pad2): track 25.5 -> 0.00 mm, vias 2 -> 0
- net +5V: track 332.5 -> 312.4 mm, vias 11 -> 9
- net Net-(J5-PadS1): track 17.0 -> 0.25 mm
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Other:
- board text removed: "+ -"
