File: Hardware/TrackJet_H01/USB.sch (KiCad schematic (older format))
At the start: 17 parts, among them J5 TYPE-C-31-M-12, Q2 S8050, Q3 S8050, U3 CH340G, Y1 12MHz

Commit message: Updated H01 PCB
Connections:
- net at Q3.1 (B), R10.1: no longer Q2.2 (E)
- net at Q2.1 (B), R9.1: no longer Q3.2 (E)
- net at R9.2, U3.13 (~DTR): now also Q3.2 (E)
- net at R10.2, U3.14 (~RTS): now also Q2.2 (E)
Other:
- moved on the sheet: R10, R9
Changed lines of the file:
@@
 L Device:R R10
 U 1 1 60194807
-P 6500 3950
-F 0 "R10" V 6700 3950 50  0000 C CNN
-F 1 "12K" V 6600 3950 50  0000 C CNN
-F 2 "Resistor_SMD:R_0603_1608Metric" V 6430 3950 50  0001 C CNN
-F 3 "~" H 6500 3950 50  0001 C CNN
-F 4 "C22790" H 6500 3950 50  0001 C CNN "LCSC"
-	1    6500 3950
+P 7150 4350
+F 0 "R10" V 7350 4350 50  0000 C CNN
+F 1 "12K" V 7250 4350 50  0000 C CNN
+F 2 "Resistor_SMD:R_0603_1608Metric" V 7080 4350 50  0001 C CNN
+F 3 "~" H 7150 4350 50  0001 C CNN
+F 4 "C22790" H 7150 4350 50  0001 C CNN "LCSC"
+	1    7150 4350
 	0    1    1    0
 $EndComp
@@
 L Device:R R9
 U 1 1 601953FB
-P 6500 3850
-F 0 "R9" V 6300 3850 50  0000 C CNN
-F 1 "12K" V 6400 3850 50  0000 C CNN
-F 2 "Resistor_SMD:R_0603_1608Metric" V 6430 3850 50  0001 C CNN
-F 3 "~" H 6500 3850 50  0001 C CNN
-F 4 "C22790" H 6500 3850 50  0001 C CNN "LCSC"
-	1    6500 3850
+P 7150 3450
+F 0 "R9" V 6950 3450 50  0000 C CNN
+F 1 "12K" V 7050 3450 50  0000 C CNN
+F 2 "Resistor_SMD:R_0603_1608Metric" V 7080 3450 50  0001 C CNN
+F 3 "~" H 7150 3450 50  0001 C CNN
+F 4 "C22790" H 7150 3450 50  0001 C CNN "LCSC"
+	1    7150 3450
 	0    1    1    0
 $EndComp
@@
 Wire Wire Line
 	7600 3650 6850 3950
-Wire Wire Line
-	6650 3950 6850 3950
 Connection ~ 6850 3950
 Wire Wire Line
 	6850 3950 6850 4350
 Wire Wire Line
-	7300 3450 6850 3450
-Wire Wire Line
 	6850 3450 6850 3850
-Wire Wire Line
-	6850 3850 6650 3850
-Wire Wire Line
-	7300 4350 6850 4350
 Wire Wire Line
 	6850 3850 7600 4150
@@
 	4200 3100 4200 3050
 NoConn ~ 3300 4350
+Wire Wire Line
+	6350 3850 6850 3850
+Wire Wire Line
+	6350 3950 6850 3950
+Wire Wire Line
+	7000 4350 6850 4350
+Wire Wire Line
+	6850 3450 7000 3450
 $EndSCHEMATC
