File: Hardware/TrackJet_H01/Motors.sch (KiCad schematic (older format))
At the start: 52 parts, among them J10 Conn_01x02, J11 Conn_01x02, J12 Conn_01x03_Male, J13 Conn_01x02, J14 Conn_01x02, J15 Conn_01x03_Male, J7 Conn_01x02, J8 Conn_01x03_Male, J9 Conn_01x02, Q6 AO3400A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

Commit message: Updated H01 PCB
Parts:
- C64, C65, C69, C70, C72, C73: value 2n2 -> 220n; LCSC C1604 -> C21120
Other:
- note added: "Sallen Key\nButterworth response\nLow Pass\n-3dB @ 5 Hz\nG = 32,33"
- note removed: "Sallen Key\nButterworth response\nLow Pass\n-3dB @ 500 Hz\nG = 32,33"
Changed lines of the file:
@@
 	5500 3300 5500 3150
 Text Notes 3500 3700 0    50   ~ 0
-Sallen Key\nButterworth response\nLow Pass\n-3dB @ 500 Hz\nG = 32,33
+Sallen Key\nButterworth response\nLow Pass\n-3dB @ 5 Hz\nG = 32,33
 Text HLabel 4350 4200 2    50   Input ~ 0
 SERVO2_CURRENT
@@
 P 3000 4350
 F 0 "C70" H 2885 4304 50  0000 R CNN
-F 1 "2n2" H 2885 4395 50  0000 R CNN
+F 1 "220n" H 2885 4395 50  0000 R CNN
 F 2 "Capacitor_SMD:C_0603_1608Metric" H 3038 4200 50  0001 C CNN
 F 3 "~" H 3000 4350 50  0001 C CNN
-F 4 "C1604" H 3000 4350 50  0001 C CNN "LCSC"
+F 4 "C21120" H 3000 4350 50  0001 C CNN "LCSC"
 	1    3000 4350
 	-1   0    0    1
@@
 P 3300 3750
 F 0 "C69" V 3048 3750 50  0000 C CNN
-F 1 "2n2" V 3139 3750 50  0000 C CNN
+F 1 "220n" V 3139 3750 50  0000 C CNN
 F 2 "Capacitor_SMD:C_0603_1608Metric" H 3338 3600 50  0001 C CNN
 F 3 "~" H 3300 3750 50  0001 C CNN
-F 4 "C1604" H 3300 3750 50  0001 C CNN "LCSC"
+F 4 "C21120" H 3300 3750 50  0001 C CNN "LCSC"
 	1    3300 3750
 	0    1    1    0
@@
 $EndComp
 Text Notes 3500 1400 0    50   ~ 0
-Sallen Key\nButterworth response\nLow Pass\n-3dB @ 500 Hz\nG = 32,33
+Sallen Key\nButterworth response\nLow Pass\n-3dB @ 5 Hz\nG = 32,33
 Text HLabel 4350 1900 2    50   Input ~ 0
 SERVO1_CURRENT
@@
 P 3000 2050
 F 0 "C65" H 2885 2004 50  0000 R CNN
-F 1 "2n2" H 2885 2095 50  0000 R CNN
+F 1 "220n" H 2885 2095 50  0000 R CNN
 F 2 "Capacitor_SMD:C_0603_1608Metric" H 3038 1900 50  0001 C CNN
 F 3 "~" H 3000 2050 50  0001 C CNN
-F 4 "C1604" H 3000 2050 50  0001 C CNN "LCSC"
+F 4 "C21120" H 3000 2050 50  0001 C CNN "LCSC"
 	1    3000 2050
 	-1   0    0    1
@@
 P 3300 1450
 F 0 "C64" V 3048 1450 50  0000 C CNN
-F 1 "2n2" V 3139 1450 50  0000 C CNN
+F 1 "220n" V 3139 1450 50  0000 C CNN
 F 2 "Capacitor_SMD:C_0603_1608Metric" H 3338 1300 50  0001 C CNN
 F 3 "~" H 3300 1450 50  0001 C CNN
-F 4 "C1604" H 3300 1450 50  0001 C CNN "LCSC"
+F 4 "C21120" H 3300 1450 50  0001 C CNN "LCSC"
 	1    3300 1450
 	0    1    1    0
@@
 	5500 5900 5500 5750
 Text Notes 3500 5900 0    50   ~ 0
-Sallen Key\nButterworth response\nLow Pass\n-3dB @ 500 Hz\nG = 32,33
+Sallen Key\nButterworth response\nLow Pass\n-3dB @ 5 Hz\nG = 32,33
 Text HLabel 4350 6400 2    50   Input ~ 0
 SERVO3_CURRENT
@@
 P 3000 6550
 F 0 "C73" H 2885 6504 50  0000 R CNN
-F 1 "2n2" H 2885 6595 50  0000 R CNN
+F 1 "220n" H 2885 6595 50  0000 R CNN
 F 2 "Capacitor_SMD:C_0603_1608Metric" H 3038 6400 50  0001 C CNN
 F 3 "~" H 3000 6550 50  0001 C CNN
-F 4 "C1604" H 3000 6550 50  0001 C CNN "LCSC"
+F 4 "C21120" H 3000 6550 50  0001 C CNN "LCSC"
 	1    3000 6550
 	-1   0    0    1
@@
 P 3300 5950
 F 0 "C72" V 3048 5950 50  0000 C CNN
-F 1 "2n2" V 3139 5950 50  0000 C CNN
+F 1 "220n" V 3139 5950 50  0000 C CNN
 F 2 "Capacitor_SMD:C_0603_1608Metric" H 3338 5800 50  0001 C CNN
 F 3 "~" H 3300 5950 50  0001 C CNN
-F 4 "C1604" H 3300 5950 50  0001 C CNN "LCSC"
+F 4 "C21120" H 3300 5950 50  0001 C CNN "LCSC"
 	1    3300 5950
 	0    1    1    0

Commit message: H01 update
Parts:
- removed C63, C67: 10u, Capacitor_SMD:C_0805_2012Metric, symbol Device:C
- removed R44, R50: 56K, Resistor_SMD:R_0603_1608Metric, symbol Device:R
- removed U16, U18: DRV8871DDA, Package_SO:Texas_HTSOP-8-1EP_3.9x4.9mm_P1.27mm_EP2.95x4.9mm_Mask2.4x3.1mm_ThermalVias, symbol Driver_Motor:DRV8871DDA
- added C23: 2u2, Capacitor_SMD:C_0603_1608Metric, symbol Device:C
- added C24: 10u, Capacitor_SMD:C_0805_2012Metric, symbol Device:C
- added C25: 10n, Capacitor_SMD:C_0603_1608Metric, symbol Device:C
- added R76, R77: R, Resistor_SMD:R_1206_3216Metric_Pad1.30x1.75mm_HandSolder, symbol Device:R
- added U22: DRV8833PWP, Package_SO:HTSSOP-16-1EP_4.4x5mm_P0.65mm_EP3.4x5mm_Mask2.46x2.31mm_ThermalVias, symbol Driver_Motor:DRV8833PWP
Connections:
- net +12V: now also C24.1, C25.1, U22.1 (nSLEEP), U22.12 (VM)
- net GND: now also C23.2, C24.2, R76.2, R77.2, U22.13 (GND), U22.17 (GND(PPAD))
- net MOTA_IN1: now also U22.9 (BIN1)
- net MOTA_IN2: now also U22.10 (BIN2)
- net MOTB_IN1: now also U22.16 (AIN1)
- net MOTB_IN2: now also U22.15 (AIN2)
- net at J7.1 (Pin_1): now also U22.7 (BOUT1)
- net at J7.2 (Pin_2): now also U22.5 (BOUT2)
- net at J9.1 (Pin_1): now also U22.2 (AOUT1)
- net at J9.2 (Pin_2): now also U22.4 (AOUT2)
- new net: C25.2, U22.11 (VCP)
- new net: C23.1, U22.14 (VINT)
- new net: R76.1, U22.3 (AISEN)
- new net: R77.1, U22.6 (BISEN)
- no-connect marks 0 -> 1
Other:
- moved on the sheet: J7, J9
