File: Hardware/TrackJet_H01/TrackJet_H01.kicad_pcb (KiCad board)
At the start: 2 copper layers, 90 x 100 mm, 205 parts, among them IC1 TP4056, J1 Conn_01x06_Female, J10 Conn_01x02, J11 Conn_01x02, J12 Conn_01x03_Male, J13 Conn_01x02, J14 Conn_01x02, J15 Conn_01x03_Male, J16 Conn_01x02_Male, J2 Conn_01x06_Female, J3 Conn_01x05_Male, J4 Conn_01x05_Male, J5 TYPE-C-31-M-12, J6 Conn_01x01_Male, J7 Conn_01x02, J8 Conn_01x03_Male, J9 Conn_01x02, Q1 2N7002, Q2 S8050, Q3 S8050, Q5 S8050, Q6 AO3400A, Q7 AO3400A, Q8 AO3400A, Q9 AO3400A, SW1 Rotary_Encoder_Switch, SW2 SW_DPST, SW3 MT-102, U1 ESP32-WROOM-32D, U10 TCRT5000, U11 TCRT5000, U12 TCRT5000, U13 74HC595, U14 74HC595, U15 CD4051B, U16 DRV8871DDA, U17 LM358, U18 DRV8871DDA, U19 LM358, U2 MPU-6050, U20 74HC595, U21 74HC595, U3 CH340G, U4 AMS1117-3.3, U5 TPS61088RHLR, U6 MT3608, U7 TCRT5000, U8 TCRT5000, U9 TCRT5000, Y1 12MHz

Commit message: Updated H01 PCB
Parts:
- removed C58: 100n, Capacitor_SMD:C_0603_1608Metric
- removed H2, H3: MountingHole, MountingHole:MountingHole_3.2mm_M3
- removed Q5: S8050, Package_TO_SOT_SMD:SOT-23
- added C22: 1u, Capacitor_SMD:C_0603_1608Metric, F.Cu at (66.4, 40.3)
- added D13: B5819W, Diode_SMD:D_SOD-123, F.Cu at (10.0, 15.7)
- added D14: LED_GREEN, LED_THT:LED_D3.0mm, F.Cu at (63.1, 36.0)
- added D15: B5819W, Diode_SMD:D_SOD-123, F.Cu at (77.9, 26.7)
- C39: value more than 1uF, footprint? -> 1u
- C41: value f -> 1n
- C64, C65, C69, C70, C72, C73: value 2n2 -> 220n
- F1: value Fuse -> Fuse 15A
- G2: renamed from .; value . -> LOGO
- R15: value R -> 24K
- R16: value R -> 150K
- R17: value R -> 200K
- R18: value R -> 240K
- R19, R28: value R -> 30K
- R23: value 3M3 -> 3M
- R24: value 51K -> 10K
- R26: value 10M -> 1K
- R27: value R -> 220K
- R30, R32, R34, R36, R38, R40: value 10K -> 1K
- moved R40 94.6 mm to (88.9, 40.4), turned to 90 degrees
- moved R75 94.0 mm to (87.3, 40.4), turned to 90 degrees
- moved C21 93.6 mm to (85.8, 40.4), turned to 90 degrees
- moved C19 84.0 mm to (82.2, 30.7)
- moved R38 84.0 mm to (82.2, 27.7)
- moved R73 84.0 mm to (82.2, 29.2)
- moved R26 62.7 mm to (62.7, 32.9), turned to 0 degrees
- moved R24 56.4 mm to (64.8, 40.3), turned to 90 degrees
- moved C20 44.5 mm to (1.91, 32.8), turned to 0 degrees
- moved R74 43.4 mm to (1.91, 34.3), turned to 180 degrees
- moved R36 42.7 mm to (2.67, 42.4), turned to 180 degrees
- moved C17 41.9 mm to (2.41, 46.5), turned to 180 degrees
- moved R71 39.2 mm to (2.41, 48.0), turned to 180 degrees
- moved R34 37.4 mm to (2.67, 40.8), turned to 180 degrees
- renumbered G*** to G1
Connections:
- C17 pad 1: /Mux Demux Matrix/Analog_IN_2 -> /Encoders/ENCODER2
- C19 pad 1: /Mux Demux Matrix/Analog_IN_4 -> /Encoders/ENCODER4
- C20 pad 1: /Mux Demux Matrix/Analog_IN_5 -> /Encoders/ENCODER5
- C21 pad 1: /Mux Demux Matrix/Analog_IN_6 -> /Encoders/ENCODER6
- C64 pad 1: /Motors/SERVO1_CURRENT -> /Mux Demux Matrix/Analog_IN_4
- C69 pad 1: /Motors/SERVO2_CURRENT -> /Mux Demux Matrix/Analog_IN_5
- C72 pad 1: /Motors/SERVO3_CURRENT -> /Mux Demux Matrix/Analog_IN_6
- Q3 pad 1: Net-(Q2-Pad2) -> Net-(Q3-Pad1)
- Q3 pad 2: Net-(Q2-Pad1) -> Net-(Q3-Pad2)
- R10 pad 1: Net-(Q2-Pad2) -> Net-(Q3-Pad1)
- R10 pad 2: Net-(R10-Pad2) -> Net-(Q2-Pad2)
- R24 pad 1: Net-(Q5-Pad3) -> +3V3
- R24 pad 2: +BATT -> /USB/ESP_RST
- R26 pad 1: /Power/5V_ENABLE -> +5V
- R26 pad 2: +BATT -> Net-(D14-Pad2)
- R48 pad 1: /Motors/SERVO1_CURRENT -> /Mux Demux Matrix/Analog_IN_4
- R54 pad 1: /Motors/SERVO2_CURRENT -> /Mux Demux Matrix/Analog_IN_5
- R63 pad 1: /Motors/SERVO3_CURRENT -> /Mux Demux Matrix/Analog_IN_6
- R71 pad 1: /Mux Demux Matrix/Analog_IN_2 -> /Encoders/ENCODER2
- R73 pad 1: /Mux Demux Matrix/Analog_IN_4 -> /Encoders/ENCODER4
- R74 pad 1: /Mux Demux Matrix/Analog_IN_5 -> /Encoders/ENCODER5
- R75 pad 1: /Mux Demux Matrix/Analog_IN_6 -> /Encoders/ENCODER6
- R9 pad 2: Net-(R9-Pad2) -> Net-(Q3-Pad2)
- SW2 pad 1: GND -> (no net)
- SW2 pad 3: (no net) -> GND
- U1 pad 27: /Power/5V_ENABLE -> /Motors/SERVO2_CTRL
- U1 pad 4: /Motors/SERVO1_CURRENT -> /Motors/SERVO3_CTRL
- U1 pad 6: /Motors/SERVO3_CURRENT -> /Encoders/ENCODER5
- U1 pad 7: /Motors/SERVO2_CURRENT -> /Encoders/ENCODER6
- U1 pad 8: /Motors/SERVO2_CTRL -> /Encoders/ENCODER2
- U1 pad 9: /Motors/SERVO3_CTRL -> /Encoders/ENCODER4
- U15 pad 14: /Mux Demux Matrix/Analog_IN_2 -> (no net)
- U17 pad 1: /Motors/SERVO2_CURRENT -> /Mux Demux Matrix/Analog_IN_5
- U17 pad 7: /Motors/SERVO1_CURRENT -> /Mux Demux Matrix/Analog_IN_4
- U19 pad 1: /Motors/SERVO3_CURRENT -> /Mux Demux Matrix/Analog_IN_6
- U3 pad 13: Net-(R9-Pad2) -> Net-(Q3-Pad2)
- U3 pad 14: Net-(R10-Pad2) -> Net-(Q2-Pad2)
- U6 pad 4: Net-(Q5-Pad3) -> +BATT
Routing:
- net /Motors/SERVO1_CURRENT: track 119.9 -> 0.00 mm, vias 10 -> 0
- net Net-(R40-Pad2): track 120.2 -> 7.04 mm, vias 7 -> 1
- net /Encoders/ENCODER6: track 0.00 -> 111.7 mm, vias 0 -> 6
- net Net-(R38-Pad2): track 118.9 -> 8.90 mm, vias 7 -> 1
- net /Power/5V_ENABLE: track 108.6 -> 0.00 mm, vias 4 -> 0
- net /Motors/SERVO2_CURRENT: track 105.8 -> 0.00 mm, vias 10 -> 0
- net /Motors/SERVO3_CURRENT: track 79.7 -> 0.00 mm, vias 8 -> 0
- net /Encoders/ENCODER5: track 0.00 -> 76.9 mm, vias 0 -> 6
- net /Encoders/ENCODER4: track 0.00 -> 70.5 mm, vias 0 -> 12
- net /Encoders/ENCODER2: track 0.00 -> 67.7 mm, vias 0 -> 8
- net +3V3: track 389.0 -> 441.9 mm, vias 10 -> 16
- net Net-(R36-Pad2): track 53.3 -> 6.61 mm, vias 6 -> 0
- net Net-(R34-Pad2): track 68.0 -> 25.5 mm, vias 4 -> 2
- net /Mux Demux Matrix/Analog_IN_4: track 6.79 -> 33.4 mm, vias 0 -> 4
- net /Mux Demux Matrix/Analog_IN_6: track 9.50 -> 36.0 mm, vias 0 -> 4
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Other:
- board text added: "+ -"

Commit message: Updated H01
Other:
- board text added: "PWR"
- board text added: "The TrackJet project designed with passion by the Vědátoři team 06-2021"
- board text added: "TrackJet_H01"
- board text removed: "SERGEJ_H00"
- board text removed: "Sergej project designed with passion by the Vědátoři team 03-2021"

Commit message: H01 update
Parts:
- removed C63, C67: 10u, Capacitor_SMD:C_0805_2012Metric
- removed R44, R50: 56K, Resistor_SMD:R_0603_1608Metric
- removed U16, U18: DRV8871DDA, Package_SO:Texas_HTSOP-8-1EP_3.9x4.9mm_P1.27mm_EP2.95x4.9mm_Mask2.4x3.1mm_ThermalVias
- added C23: 2u2, Capacitor_SMD:C_0603_1608Metric, F.Cu at (68.7, 92.6)
- added C24: 10u, Capacitor_SMD:C_0805_2012Metric, F.Cu at (66.2, 92.3)
- added C25: 10n, Capacitor_SMD:C_0603_1608Metric, F.Cu at (63.5, 92.6)
- added R76: R, Resistor_SMD:R_1206_3216Metric_Pad1.30x1.75mm_HandSolder, B.Cu at (63.2, 80.0)
- added R77: R, Resistor_SMD:R_1206_3216Metric_Pad1.30x1.75mm_HandSolder, B.Cu at (61.6, 83.9)
- added U22: DRV8833PWP, Package_SO:HTSSOP-16-1EP_4.4x5mm_P0.65mm_EP3.4x5mm_Mask2.46x2.31mm_ThermalVias, F.Cu at (66.0, 86.4)
- moved G2 49.3 mm to (77.3, 48.8), turned to 90 degrees
Routing:
- net Net-(J7-Pad2): track 5.64 -> 115.3 mm
- net Net-(J7-Pad1): track 10.1 -> 119.1 mm
- net +12V: track 201.2 -> 136.3 mm
- net /Motors/MOTB_IN1: track 114.1 -> 51.8 mm, vias 6 -> 2
- net /Motors/MOTB_IN2: track 95.1 -> 49.2 mm, vias 4 -> 2
- net Net-(J9-Pad1): track 6.13 -> 51.9 mm, vias 0 -> 2
- net Net-(J9-Pad2): track 10.5 -> 52.2 mm, vias 0 -> 2
- net /Motors/MOTA_IN2: track 80.9 -> 46.0 mm, vias 8 -> 4
- net GND: track 161.6 -> 147.2 mm, vias 133 -> 129
- net /Motors/MOTA_IN1: track 60.8 -> 47.9 mm
- net /Mux Demux Matrix/Analog_IN_7: track 145.7 -> 139.0 mm
- net Net-(R76-Pad1): track 0.00 -> 5.16 mm, vias 0 -> 1
- net Net-(R77-Pad1): track 0.00 -> 5.08 mm, vias 0 -> 1
- net /Motors/SERVO3_CTRL: track 85.7 -> 81.6 mm
- net Net-(C23-Pad1): track 0.00 -> 3.84 mm
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
Commit message: H01 update
Parts:
- moved R77 8.35 mm to (65.5, 76.6), turned to 90 degrees
- moved R76 7.85 mm to (70.9, 78.1), turned to 0 degrees
Routing:
- net Net-(J9-Pad1): track 51.9 -> 54.3 mm
- net Net-(R76-Pad1): track 5.16 -> 6.93 mm
- net Net-(R77-Pad1): track 5.08 -> 5.98 mm

Commit message: H01 update
Other:
- board text added: "+ - MOT 6"
- board text added: "MOT 2"
- board text removed: "+ - MOT 2"
- board text removed: "MOT 0"

Commit message: H01 update
Other:
- board text added: "LINE LEFT LINE RIGHT"
- board text added: "PWM 5V GND"
- board text removed: "GND 5V PWM"

Commit message: Update TrackJet_H01.kicad_pcb
Other:
- board text added: "LINE RIGHT LINE LEFT"
- board text added: "www.github.com/vedatori/TrackJet"
- board text removed: "LINE LEFT LINE RIGHT"
